File: hardware/6507 SBC.kicad_sch (KiCad schematic)
At the start: 21 parts

Commit message: Added license and PDF schematic
Other:
- company: (none) -> Anders B. Nielsen
- title: (none) -> Single Breadboard Computer
Changed lines of the file:
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@@
 (kicad_sch (version 20211123) (generator eeschema)
   (paper "A4")
+  (title_block
+    (title "Single Breadboard Computer")
+    (rev "0")
+    (company "Anders B. Nielsen")
+    (comment 1 "License: https://creativecommons.org/licenses/by-nc/4.0/legalcode")
+  )
   (junction (at 119.38 54.61) (diameter 0) (color 0 0 0 0)
   )
